File: pcb/pcb.kicad_pcb (KiCad board)
At the start: 2 copper layers, 114.3 x 57.2 mm, 57 parts, among them J1 USB_C_Receptacle_USB2.0, J2 SWD, SW1 SW_Push, U1 W25Q128JVS, U2 USBLC6-2SC6, U3 RP2040, U4 XC6206PxxxMR-Regulator_Linear, Y1 12MHz

Commit message: Update readme
Parts:
- moved D5 16.2 mm to (113.8, 102.9)
- moved D10 14.7 mm to (80.8, 121.4), turned to 180 degrees
Routing:
- net /ROW1: track 100.7 -> 88.3 mm
- net Net-(D10-A): track 18.0 -> 10.6 mm
- net Net-(D5-A): track 18.0 -> 12.4 mm
- net /ROW0: track 136.4 -> 138.5 mm
Other:
- board text added: "rmk by dcpedit (rev 2) github.com/dcpedit/rmk"
- board text removed: "rmk by dcpedit (rev 1) github.com/dcpedit/rmk"
Changed lines of the file:
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@@
         (effects (font (size 1 1) (thickness 0.15)))
     )
-    (fp_text value "SW_Push" (at 52.784375 94.591 90) (layer "F.Fab")
+    (fp_text value "SW_Push" (at 52.784375 94.591 90) (layer "F.Fab") hide
         (effects (font (size 1 1) (thickness 0.15)))
     )
@@
   )
   (footprint "Diode_SMD:D_SOD-123" (layer "B.Cu")
-    (at 84.1375 135.73125 90)
+    (at 80.773 121.412 180)
     (descr "SOD-123")
     (tags "SOD-123")
@@
     (property "ki_keywords" "diode")
     (attr smd)
-    (fp_text reference "D10" (at -0.00635 -2.0447 90) (layer "B.SilkS")
+    (fp_text reference "D10" (at -0.00635 -2.0447) (layer "B.SilkS")
         (effects (font (size 1 1) (thickness 0.15)) (justify mirror))
     )
-    (fp_text value "D" (at 0 -2.1 90) (layer "B.Fab")
+    (fp_text value "D" (at 0 -2.1) (layer "B.Fab")
         (effects (font (size 1 1) (thickness 0.15)) (justify mirror))
     )
-    (fp_text user "${REFERENCE}" (at 0 2 90) (layer "B.Fab")
+    (fp_text user "${REFERENCE}" (at 0 2) (layer "B.Fab")
         (effects (font (size 1 1) (thickness 0.15)) (justify mirror))
     )
@@
     (fp_line (start 1.4 0.9) (end 1.4 -0.9)
       (stroke (width 0.1) (type solid)) (layer "B.Fab"))
-    (pad "1" smd roundrect (at -1.65 0 90) (size 0.9 1.2) (layers "B.Cu" "B.Paste" "B.Mask") (roundrect_rratio 0.25)
+    (pad "1" smd roundrect (at -1.65 0 180) (size 0.9 1.2) (layers "B.Cu" "B.Paste" "B.Mask") (roundrect_rratio 0.25)
       (net 40 "/ROW1") (pinfunction "K") (pintype "passive"))
-    (pad "2" smd roundrect (at 1.65 0 90) (size 0.9 1.2) (layers "B.Cu" "B.Paste" "B.Mask") (roundrect_rratio 0.25)
+    (pad "2" smd roundrect (at 1.65 0 180) (size 0.9 1.2) (layers "B.Cu" "B.Paste" "B.Mask") (roundrect_rratio 0.25)
       (net 38 "Net-(D10-A)") (pinfunction "A") (pintype "passive"))
     (model "${KICAD6_3DMODEL_DIR}/Diode_SMD.3dshapes/D_SOD-123.wrl"
@@
   )
   (footprint "Diode_SMD:D_SOD-123" (layer "B.Cu")
-    (at 129.38125 107.15625 90)
+    (at 113.792 102.87 90)
     (descr "SOD-123")
     (tags "SOD-123")
@@
     (effects (font (size 1 1) (thickness 0.15)))
   )
-  (gr_text "rmk by dcpedit (rev 1)\ngithub.com/dcpedit/rmk" (at 54.5084 133.604) (layer "B.SilkS")
+  (gr_text "rmk by dcpedit (rev 2)\ngithub.com/dcpedit/rmk" (at 54.5084 133.604) (layer "B.SilkS")
     (effects (font (size 1.5 1.5) (thickness 0.3) bold) (justify left bottom mirror))
   )
@@
   (segment (start 93.0275 88.32875) (end 94.2375 87.11875) (width 0.2) (layer "B.Cu") (net 32))
   (segment (start 93.0275 90.32875) (end 93.0275 88.32875) (width 0.2) (layer "B.Cu") (net 32))
-  (segment (start 126.88625 103.01125) (end 129.38125 105.50625) (width 0.2) (layer "B.Cu") (net 33))
+  (segment (start 119.22125 99.85375) (end 115.15825 99.85375) (width 0.2) (layer "B.Cu") (net 33))
   (segment (start 120.43125 98.64375) (end 120.43125 96.64375) (width 0.2) (layer "B.Cu") (net 33))
   (segment (start 122.88125 96.64375) (end 123.03125 96.49375) (width 0.2) (layer "B.Cu") (net 33))
-  (segment (start 123.03125 96.49375) (end 123.03125 98.031338) (width 0.2) (layer "B.Cu") (net 33))
-  (segment (start 123.03125 98.031338) (end 126.88625 101.886338) (width 0.2) (layer "B.Cu") (net 33))
+  (segment (start 115.15825 99.85375) (end 113.792 101.22) (width 0.2) (layer "B.Cu") (net 33))
   (segment (start 120.43125 96.64375) (end 122.88125 96.64375) (width 0.2) (layer "B.Cu") (net 33))
-  (segment (start 126.88625 101.886338) (end 126.88625 103.01125) (width 0.2) (layer "B.Cu") (net 33))
   (segment (start 119.22125 99.85375) (end 120.43125 98.64375) (width 0.2) (layer "B.Cu") (net 33))
   (segment (start 39.90625 115.66875) (end 41.11625 114.45875) (width 0.2) (layer "B.Cu") (net 34))
@@
   (segment (start 105.455 111.743241) (end 105.455 112.53625) (width 0.2) (layer "B.Cu") (net 37))
   (segment (start 97.79 109.37875) (end 97.79 107.37875) (width 0.2) (layer "B.Cu") (net 37))
-  (segment (start 81.2292 131.17295) (end 84.1375 134.08125) (width 0.2) (layer "B.Cu") (net 38))
   (segment (start 75.21925 125.21875) (end 77.66925 125.21875) (width 0.2) (layer "B.Cu") (net 38))
   (segment (start 77.66925 125.21875) (end 77.81925 125.06875) (width 0.2) (layer "B.Cu") (net 38))
-  (segment (start 81.2292 130.348191) (end 81.2292 131.17295) (width 0.2) (layer "B.Cu") (net 38))
+  (segment (start 77.81925 122.71575) (end 79.123 121.412) (width 0.2) (layer "B.Cu") (net 38))
   (segment (start 74.00925 128.42875) (end 74.00925 126.42875) (width 0.2) (layer "B.Cu") (net 38))
-  (segment (start 77.81925 125.06875) (end 77.81925 126.938241) (width 0.2) (layer "B.Cu") (net 38))
-  (segment (start 77.81925 126.938241) (end 81.2292 130.348191) (width 0.2) (layer "B.Cu") (net 38))
+  (segment (start 77.81925 125.06875) (end 77.81925 122.71575) (width 0.2) (layer "B.Cu") (net 38))
   (segment (start 74.00925 126.42875) (end 75.21925 125.21875) (width 0.2) (layer "B.Cu") (net 38))
   (segment (start 94.3356 99.28125) (end 94.3356 118.48045) (width 0.2) (layer "F.Cu") (net 39))
@@
   (via (at 113.662518 118.08175) (size 0.6) (drill 0.3) (layers "F.Cu" "B.Cu") (net 39))
   (segment (start 41.275 99.28125) (end 65.0875 99.28125) (width 0.2) (layer "B.Cu") (net 39))
-  (segment (start 129.38125 108.80625) (end 121.21615 108.80625) (width 0.2) (layer "B.Cu") (net 39))
   (segment (start 113.662518 118.08175) (end 113.862018 118.28125) (width 0.2) (layer "B.Cu") (net 39))
   (segment (start 115.225884 118.28125) (end 115.642517 118.697883) (width 0.2) (layer "B.Cu") (net 39))
   (segment (start 103.720315 117.93125) (end 106.934 117.93125) (width 0.2) (layer "B.Cu") (net 39))
+  (segment (start 118.871 104.52) (end 121.158 106.807) (width 0.2) (layer "B.Cu") (net 39))
   (segment (start 107.31405 117.5512) (end 108.512412 117.5512) (width 0.2) (layer "B.Cu") (net 39))
   (segment (start 65.0875 99.28125) (end 84.1375 99.28125) (width 0.2) (layer "B.Cu") (net 39))
-  (segment (start 121.21615 108.80625) (end 121.158 108.8644) (width 0.2) (layer "B.Cu") (net 39))
   (segment (start 109.242462 118.28125) (end 113.463018 118.28125) (width 0.2) (layer "B.Cu") (net 39))
   (segment (start 108.512412 117.5512) (end 109.242462 118.28125) (width 0.2) (layer "B.Cu") (net 39))
@@
   (segment (start 106.934 117.93125) (end 107.31405 117.5512) (width 0.2) (layer "B.Cu") (net 39))
   (segment (start 94.3864 118.53125) (end 94.5859 118.73075) (width 0.2) (layer "B.Cu") (net 39))
+  (segment (start 121.158 106.807) (end 121.158 108.8644) (width 0.2) (layer "B.Cu") (net 39))
+  (segment (start 113.792 104.52) (end 118.871 104.52) (width 0.2) (layer "B.Cu") (net 39))
   (segment (start 120.083 123.138366) (end 120.083 125.8435) (width 0.2) (layer "B.Cu") (net 39))
   (segment (start 102.920814 118.73075) (end 103.720315 117.93125) (width 0.2) (layer "B.Cu") (net 39))
-  (segment (start 84.1756 135.8392) (end 84.54425 135.47055) (width 0.2) (layer "F.Cu") (net 40))
-  (segment (start 84.54425 124.19295) (end 88.8492 119.888) (width 0.2) (layer "F.Cu") (net 40))
-  (segment (start 84.54425 135.47055) (end 84.54425 124.19295) (width 0.2) (layer "F.Cu") (net 40))
+  (segment (start 83.947 121.412) (end 87.3252 121.412) (width 0.2) (layer "F.Cu") (net 40))
+  (segment (start 87.3252 121.412) (end 88.8492 119.888) (width 0.2) (layer "F.Cu") (net 40))
   (via (at 88.8492 119.888) (size 0.6) (drill 0.3) (layers "F.Cu" "B.Cu") (net 40))
-  (via (at 84.1756 135.8392) (size 0.6) (drill 0.3) (layers "F.Cu" "B.Cu") (net 40))
+  (via (at 83.947 121.412) (size 0.6) (drill 0.3) (layers "F.Cu" "B.Cu") (net 40))
   (segment (start 103.886 118.33125) (end 107.95 118.33125) (width 0.2) (layer "B.Cu") (net 40))
   (segment (start 115.060199 118.68125) (end 119.683 123.304051) (width 0.2) (layer "B.Cu") (net 40))
   (segment (start 103.0865 119.13075) (end 103.886 118.33125) (width 0.2) (layer "B.Cu") (net 40))
-  (segment (start 84.1375 135.8773) (end 84.1756 135.8392) (width 0.2) (layer "B.Cu") (net 40))
+  (segment (start 82.423 121.412) (end 83.947 121.412) (width 0.2) (layer "B.Cu") (net 40))
   (segment (start 45.24375 118.33125) (end 69.85 118.33125) (width 0.2) (layer "B.Cu") (net 40))
   (segment (start 89.6995 119.13075) (end 103.0865 119.13075) (width 0.2) (layer "B.Cu") (net 40))
   (segment (start 69.85 118.33125) (end 88.9 118.33125) (width 0.2) (layer "B.Cu") (net 40))
-  (segment (start 84.1375 137.38125) (end 84.1375 135.8773) (width 0.2) (layer "B.Cu") (net 40))
   (segment (start 88.8492 118.38205) (end 88.9 118.33125) (width 0.2) (layer "B.Cu") (net 40))
   (segment (start 107.95 118.33125) (end 108.3 118.68125) (width 0.2) (layer "B.Cu") (net 40))
